File: homespan_test_without_homing/Hardware/Hardware.kicad_sch (KiCad schematic)
At the start: 25 parts

Commit message: add hardware
Parts:
- removed J?: end_con, symbol Connector_Generic:Conn_01x03
- added C10: 22uF, Capacitor_SMD:C_0805_2012Metric, symbol Device:C
- added C2: 4.7uF, Capacitor_SMD:C_0805_2012Metric, symbol Device:C
- added C9: 0.47uF, Capacitor_SMD:C_0805_2012Metric, symbol Device:C
- added D1: LED green, LED_SMD:LED_0603_1608Metric, symbol Device:LED
- added H1, H2, H3, H4: MountingHole, MountingHole:MountingHole_3.2mm_M3, symbol Mechanical:MountingHole
- added IC2: LT3973EDD-3.3#PBF, SamacSys_Parts:SON50P300X300X80-11N-D, symbol SamacSys_Parts:LT3973EDD-3.3#PBF
- added J1: Vin 5-40V, Connector_JST:JST_XH_B2B-XH-A_1x02_P2.50mm_Vertical, symbol Connector_Generic:Conn_01x02
- added L1: 15uH, Inductor_SMD:L_0805_2012Metric, symbol Device:L
- added R10: 12k, Resistor_SMD:R_0603_1608Metric, symbol Device:R
- added R11: 100k, Resistor_SMD:R_0603_1608Metric, symbol Device:R
- added R3: 215k, Resistor_SMD:R_0603_1608Metric, symbol Device:R
- added R7: 110, Resistor_SMD:R_0603_1608Metric, symbol Device:R
- added R9: 33k, Resistor_SMD:R_0603_1608Metric, symbol Device:R
- added SW2: SW_Push, Button_Switch_SMD:SW_SPST_B3U-1000P-B, symbol Switch:SW_Push
- C1: renamed from C?; value 22nF/50V -> 22nF/50V; footprint (none) -> Capacitor_SMD:C_0805_2012Metric
- C11, C12, C13, C14, C15, C3, C4, C5, C6, C7, C8: renamed from C?; footprint (none) -> Capacitor_SMD:C_0805_2012Metric
- IC1: renamed from IC?; footprint ESP32S3WROOM1N4R2 -> SamacSys_Parts:ESP32S3WROOM1N4R2
- IC3: renamed from IC?; footprint QFN50P500X500X90-29N -> SamacSys_Parts:QFN50P500X500X90-29N
- J2: renamed from J?; footprint (none) -> Connector_JST:JST_XH_B4B-XH-A_1x04_P2.50mm_Vertical
- J3: renamed from J?; footprint (none) -> Connector_PinHeader_2.54mm:PinHeader_1x02_P2.54mm_Vertical
- R1, R2: renamed from R?; footprint (none) -> Resistor_SMD:R_2010_5025Metric
- R4, R5, R6, R8: renamed from R?; footprint (none) -> Resistor_SMD:R_0603_1608Metric
- RV1: renamed from RV?; value R_Potentiometer -> 20k; footprint (none) -> Potentiometer_SMD:Potentiometer_ACP_CA6-VSMD_Vertical_Hole
- SW1: renamed from SW?; footprint (none) -> Button_Switch_SMD:SW_SPST_B3U-1000P-B
Connections:
- net +3V3: now also C10.2, IC2.1 (FB/VOUT), IC2.2 (OUT), IC2.8 (BD), L1.2, R7.2
- net ADC_battery: now also R10.1, R11.1, R9.2
- net GND: now also C10.1, C2.1, IC2.11 (GND_2), IC2.5 (GND_1), J1.1 (Pin_1), R10.2, R11.2, R3.2, SW2.2
- net HK-button: now also SW2.1
- net HK_led: now also D1.1 (K)
- net VS_input: now also C2.2, IC2.3 (EN/UVLO), IC2.4 (VIN), J1.2 (Pin_2), R9.1
- net end_switch: no longer names the net of IC1.23 (IO21)
- new net: D1.2 (A), R7.1
- new net: IC2.10 (RT), R3.1
- new net: C9.2, IC2.6 (SW), L1.1
- new net: C9.1, IC2.7 (BOOST)
- no-connect marks 4 -> 28
Other:
- note added: "ESP32"
- note added: "HomeKit controll"
- note added: "Motor driver"
- note added: "Mounting holes"
- note added: "Power supply"
- note added: "To read the battery level in percent. WHEN IN USE MAX Vin is 12V"
- moved on the sheet: C13, SW1

Commit message: add board
Parts:
- removed C5: 1uF/50V, Capacitor_SMD:C_0805_2012Metric, symbol Device:C
- SW1: value SW_Push -> reset
- SW2: value SW_Push -> homekit
- renumbered C6 to C5, C7 to C6
Other:
- moved on the sheet: C5, C6
Changed lines of the file:
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@@
   (junction (at 70.485 174.625) (diameter 0) (color 0 0 0 0)
   )
-  (junction (at 23.495 91.44) (diameter 0) (color 0 0 0 0)
+  (junction (at 34.925 91.44) (diameter 0) (color 0 0 0 0)
+  )
+  (junction (at 27.305 91.44) (diameter 0) (color 0 0 0 0)
   )
   (junction (at 79.375 67.945) (diameter 0) (color 0 0 0 0)
@@
   (junction (at 267.335 74.93) (diameter 0) (color 0 0 0 0)
   )
-  (junction (at 38.735 91.44) (diameter 0) (color 0 0 0 0)
-  )
   (junction (at 221.615 31.75) (diameter 0) (color 0 0 0 0)
   )
@@
   (junction (at 267.335 80.01) (diameter 0) (color 0 0 0 0)
   )
-  (junction (at 34.925 101.6) (diameter 0) (color 0 0 0 0)
-  )
   (junction (at 203.835 70.485) (diameter 0) (color 0 0 0 0)
   )
-  (junction (at 27.305 110.49) (diameter 0) (color 0 0 0 0)
+  (junction (at 27.305 100.33) (diameter 0) (color 0 0 0 0)
   )
   (junction (at 78.105 164.465) (diameter 0) (color 0 0 0 0)
@@
   (junction (at 224.155 59.69) (diameter 0) (color 0 0 0 0)
   )
-  (junction (at 34.925 110.49) (diameter 0) (color 0 0 0 0)
-  )
-  (junction (at 27.305 101.6) (diameter 0) (color 0 0 0 0)
+  (junction (at 34.925 100.33) (diameter 0) (color 0 0 0 0)
   )
   (junction (at 254.635 135.255) (diameter 0) (color 0 0 0 0)
@@
     (stroke (width 0) (type default) (color 0 0 0 0))
   )
-  (polyline (pts (xy 120.015 123.825) (xy 13.97 123.825))
+  (polyline (pts (xy 120.015 113.03) (xy 13.97 113.03))
     (stroke (width 0) (type default) (color 0 0 0 0))
   )
@@
     (stroke (width 0) (type default) (color 0 0 0 0))
   )
-  (wire (pts (xy 27.305 110.49) (xy 27.305 119.38))
+  (wire (pts (xy 27.305 100.33) (xy 27.305 109.22))
     (stroke (width 0) (type default) (color 0 0 0 0))
   )
@@
     (stroke (width 0) (type default) (color 0 0 0 0))
   )
-  (wire (pts (xy 27.305 101.6) (xy 27.305 110.49))
+  (wire (pts (xy 27.305 91.44) (xy 27.305 100.33))
     (stroke (width 0) (type default) (color 0 0 0 0))
   )
@@
     (stroke (width 0) (type default) (color 0 0 0 0))
   )
-  (wire (pts (xy 38.735 101.6) (xy 34.925 101.6))
-    (stroke (width 0) (type default) (color 0 0 0 0))
-  )
   (wire (pts (xy 97.79 55.245) (xy 99.695 55.245))
     (stroke (width 0) (type default) (color 0 0 0 0))
@@
     (stroke (width 0) (type default) (color 0 0 0 0))
   )
-  (polyline (pts (xy 120.015 13.97) (xy 120.015 123.825))
+  (polyline (pts (xy 120.015 13.97) (xy 120.015 113.03))
     (stroke (width 0) (type default) (color 0 0 0 0))
   )
@@
     (stroke (width 0) (type default) (color 0 0 0 0))
   )
-  (wire (pts (xy 23.495 91.44) (xy 23.495 101.6))
-    (stroke (width 0) (type default) (color 0 0 0 0))
-  )
   (polyline (pts (xy 195.58 111.125) (xy 195.58 133.35))
     (stroke (width 0) (type default) (color 0 0 0 0))
@@
     (stroke (width 0) (type default) (color 0 0 0 0))
   )
-  (wire (pts (xy 34.925 110.49) (xy 34.925 119.38))
+  (wire (pts (xy 34.925 100.33) (xy 34.925 109.22))
     (stroke (width 0) (type default) (color 0 0 0 0))
   )
@@
     (stroke (width 0) (type default) (color 0 0 0 0))
   )
-  (wire (pts (xy 34.925 101.6) (xy 34.925 110.49))
+  (wire (pts (xy 34.925 91.44) (xy 34.925 100.33))
     (stroke (width 0) (type default) (color 0 0 0 0))
   )
@@
     (stroke (width 0) (type default) (color 0 0 0 0))
   )
-  (polyline (pts (xy 13.97 13.97) (xy 13.97 123.825))
+  (polyline (pts (xy 13.97 13.97) (xy 13.97 113.03))
     (stroke (width 0) (type default) (color 0 0 0 0))
   )
@@
     (stroke (width 0) (type default) (color 0 0 0 0))
   )
-  (wire (pts (xy 23.495 101.6) (xy 27.305 101.6))
-    (stroke (width 0) (type default) (color 0 0 0 0))
-  )
   (wire (pts (xy 78.105 164.465) (xy 78.105 176.53))
     (stroke (width 0) (type default) (color 0 0 0 0))
@@
   )
   (wire (pts (xy 229.235 85.09) (xy 234.315 85.09))
-    (stroke (width 0) (type default) (color 0 0 0 0))
-  )
-  (wire (pts (xy 38.735 91.44) (xy 38.735 101.6))
     (stroke (width 0) (type default) (color 0 0 0 0))
   )
@@
     (pin "2")
   )
-  (symbol (lib_id "Device:C") (at 31.115 110.49 270) (unit 1)
-    (in_bom yes) (on_board yes)
-    (property "Reference" "C6" (id 0) (at 29.845 105.41 90)
-      (effects (font (size 1.27 1.27)) (justify left))
-    )
-    (property "Value" "1uF/50V" (id 1) (at 27.305 107.315 90)
-      (effects (font (size 1.27 1.27)) (justify left))
-    )
-    (property "Footprint" "Capacitor_SMD:C_0805_2012Metric" (id 2) (at 27.305 111.4552 0)
-      (effects (font (size 1.27 1.27)) hide)
-    )
-    (property "Datasheet" "~" (id 3) (at 31.115 110.49 0)
+  (symbol (lib_id "Device:C") (at 31.115 100.33 270) (unit 1)
+    (in_bom yes) (on_board yes)
+    (property "Reference" "C5" (id 0) (at 29.845 95.25 90)
+      (effects (font (size 1.27 1.27)) (justify left))
+    )
+    (property "Value" "1uF/50V" (id 1) (at 27.305 97.155 90)
+      (effects (font (size 1.27 1.27)) (justify left))
+    )
+    (property "Footprint" "Capacitor_SMD:C_0805_2012Metric" (id 2) (at 27.305 101.2952 0)
+      (effects (font (size 1.27 1.27)) hide)
+    )
+    (property "Datasheet" "~" (id 3) (at 31.115 100.33 0)
       (effects (font (size 1.27 1.27)) hide)
     )
@@
     (pin "1")
   )
-  (symbol (lib_id "Device:C") (at 31.115 101.6 270) (unit 1)
-    (in_bom yes) (on_board yes)
-    (property "Reference" "C5" (id 0) (at 29.845 96.52 90)
-      (effects (font (size 1.27 1.27)) (justify left))
-    )
-    (property "Value" "1uF/50V" (id 1) (at 27.305 98.425 90)
-      (effects (font (size 1.27 1.27)) (justify left))
-    )
-    (property "Footprint" "Capacitor_SMD:C_0805_2012Metric" (id 2) (at 27.305 102.5652 0)
-      (effects (font (size 1.27 1.27)) hide)
-    )
-    (property "Datasheet" "~" (id 3) (at 31.115 101.6 0)
-      (effects (font (size 1.27 1.27)) hide)
-    )
-    (pin "1")
-    (pin "2")
-  )
   (symbol (lib_id "power:GND") (at 79.375 78.105 0) (unit 1)
     (in_bom yes) (on_board yes) (fields_autoplaced)
@@
     (in_bom yes) (on_board yes)
     (property "Reference" "SW2" (id 0) (at 214.63 129.54 0))
-    (property "Value" "SW_Push" (id 1) (at 214.63 131.445 0))
+    (property "Value" "homekit" (id 1) (at 214.63 131.445 0))
     (property "Footprint" "Button_Switch_SMD:SW_SPST_B3U-1000P-B" (id 2) (at 214.63 122.555 0)
       (effects (font (size 1.27 1.27)) hide)
@@
     )
   )
-  (symbol (lib_id "Device:C") (at 31.115 119.38 270) (unit 1)
-    (in_bom yes) (on_board yes)
-    (property "Reference" "C7" (id 0) (at 29.845 114.3 90)
-      (effects (font (size 1.27 1.27)) (justify left))
-    )
-    (property "Value" "1uF/50V" (id 1) (at 27.305 116.205 90)
-      (effects (font (size 1.27 1.27)) (justify left))
-    )
-    (property "Footprint" "Capacitor_SMD:C_0805_2012Metric" (id 2) (at 27.305 120.3452 0)
-      (effects (font (size 1.27 1.27)) hide)
-    )
-    (property "Datasheet" "~" (id 3) (at 31.115 119.38 0)
+  (symbol (lib_id "Device:C") (at 31.115 109.22 270) (unit 1)
+    (in_bom yes) (on_board yes)
+    (property "Reference" "C6" (id 0) (at 29.845 104.14 90)
+      (effects (font (size 1.27 1.27)) (justify left))
+    )
+    (property "Value" "1uF/50V" (id 1) (at 27.305 106.045 90)
+      (effects (font (size 1.27 1.27)) (justify left))
+    )
+    (property "Footprint" "Capacitor_SMD:C_0805_2012Metric" (id 2) (at 27.305 110.1852 0)
+      (effects (font (size 1.27 1.27)) hide)
+    )
+    (property "Datasheet" "~" (id 3) (at 31.115 109.22 0)
       (effects (font (size 1.27 1.27)) hide)
     )
@@
     (in_bom yes) (on_board yes) (fields_autoplaced)
     (property "Reference" "SW1" (id 0) (at 208.915 62.865 0))
-    (property "Value" "SW_Push" (id 1) (at 208.915 65.405 0))
+    (property "Value" "reset" (id 1) (at 208.915 65.405 0))
     (property "Footprint" "Button_Switch_SMD:SW_SPST_B3U-1000P-B" (id 2) (at 208.915 65.405 0)
       (effects (font (size 1.27 1.27)) hide)
@@
       (reference "C4") (unit 1) (value "100nF/50V") (footprint "Capacitor_SMD:C_0805_2012Metric")
     )
-    (path "/7c9b5afd-5e5f-4d90-bcd4-d9953f392e6e"
+    (path "/3dfc3f84-612d-4bde-9ead-8bc1d9be7938"
       (reference "C5") (unit 1) (value "1uF/50V") (footprint "Capacitor_SMD:C_0805_2012Metric")
     )
-    (path "/3dfc3f84-612d-4bde-9ead-8bc1d9be7938"
+    (path "/b59ab2df-297a-4856-965d-56f4c6d84ea6"
       (reference "C6") (unit 1) (value "1uF/50V") (footprint "Capacitor_SMD:C_0805_2012Metric")
-    )
-    (path "/b59ab2df-297a-4856-965d-56f4c6d84ea6"
-      (reference "C7") (unit 1) (value "1uF/50V") (footprint "Capacitor_SMD:C_0805_2012Metric")
     )
     (path "/3716de76-480f-419e-88f4-bed7bf6dd927"
@@
     )
     (path "/f7fdc9f1-357e-4038-b29d-627e22c6d89a"
-      (reference "SW1") (unit 1) (value "SW_Push") (footprint "Button_Switch_SMD:SW_SPST_B3U-1000P-B")
+      (reference "SW1") (unit 1) (value "reset") (footprint "Button_Switch_SMD:SW_SPST_B3U-1000P-B")
     )
     (path "/a435c017-fb7c-4cc4-9f13-037fc134fbd2"
-      (reference "SW2") (unit 1) (value "SW_Push") (footprint "Button_Switch_SMD:SW_SPST_B3U-1000P-B")
-    )
-  )
+      (reference "SW2") (unit 1) (value "homekit") (footprint "Button_Switch_SMD:SW_SPST_B3U-1000P-B")
+    )
+  )
