File: homespan_test_without_homing/Hardware/_autosave-Hardware.kicad_pcb (KiCad board)
At the start: 2 copper layers, 41 x 41 mm, 40 parts, among them IC1 ESP32-S3-WROOM-1-N4R2, IC2 LT3973EDD-3.3#PBF, IC3 TMC2209-LA, J1 Vin 5-40V, J2 motor_con, J3 boot, SW1 reset, SW2 homekit

Commit message: add board
Changed lines of the file:
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@@
   )
   (paper "A4")
+  (title_block
+    (comment 4 "AISLER Project ID: RAMMTZQH")
+  )
   (layers
     (0 "F.Cu" signal)
@@
       (outputformat 1)
       (mirror false)
-      (drillshape 1)
+      (drillshape 0)
       (scaleselection 1)
-      (outputdirectory "")
+      (outputdirectory "gerber/")
     )
   )
@@
     (fp_line (start 0 -1.35) (end 0.625 -2.35) (layer "F.Fab") (width 0.1))
     (fp_line (start 9.95 -2.35) (end -2.45 -2.35) (layer "F.Fab") (width 0.1))
-    (pad "1" thru_hole roundrect (at 0 0 90) (size 1.7 1.95) (drill 0.95) (layers *.Cu *.Mask) (roundrect_rratio 0.147059)
+    (pad "1" thru_hole roundrect (at 0 0 90) (size 1.7 1.95) (drill 0.95) (layers *.Cu *.Mask) (roundrect_rratio 0.1470588235)
       (net 49 "/B2") (pinfunction "Pin_1") (pintype "passive"))
     (pad "2" thru_hole oval (at 2.5 0 90) (size 1.7 1.95) (drill 0.95) (layers *.Cu *.Mask)
@@
     (fp_line (start -0.625 -2.35) (end 0 -1.35) (layer "F.Fab") (width 0.1))
     (fp_line (start 0 -1.35) (end 0.625 -2.35) (layer "F.Fab") (width 0.1))
-    (pad "1" thru_hole roundrect (at 0 0 270) (size 1.7 2) (drill 1) (layers *.Cu *.Mask) (roundrect_rratio 0.147059)
+    (pad "1" thru_hole roundrect (at 0 0 270) (size 1.7 2) (drill 1) (layers *.Cu *.Mask) (roundrect_rratio 0.1470588235)
       (net 3 "GND") (pinfunction "Pin_1") (pintype "passive"))
     (pad "2" thru_hole oval (at 2.5 0 270) (size 1.7 2) (drill 1) (layers *.Cu *.Mask)
@@
     (fp_line (start 2.5 1.25) (end 2.5 -1.25) (layer "B.Fab") (width 0.1))
     (fp_line (start -2.5 1.25) (end 2.5 1.25) (layer "B.Fab") (width 0.1))
-    (pad "1" smd roundrect (at -2.3125 0 90) (size 1.225 2.65) (layers "B.Cu" "B.Paste" "B.Mask") (roundrect_rratio 0.204082)
+    (pad "1" smd roundrect (at -2.3125 0 90) (size 1.225 2.65) (layers "B.Cu" "B.Paste" "B.Mask") (roundrect_rratio 0.2040816327)
       (net 57 "Net-(IC3-Pad23)") (pintype "passive"))
-    (pad "2" smd roundrect (at 2.3125 0 90) (size 1.225 2.65) (layers "B.Cu" "B.Paste" "B.Mask") (roundrect_rratio 0.204082)
+    (pad "2" smd roundrect (at 2.3125 0 90) (size 1.225 2.65) (layers "B.Cu" "B.Paste" "B.Mask") (roundrect_rratio 0.2040816327)
       (net 3 "GND") (pintype "passive"))
     (model "${KICAD6_3DMODEL_DIR}/Resistor_SMD.3dshapes/R_2010_5025Metric.wrl"
@@
     (fp_line (start 2.5 -1.25) (end -2.5 -1.25) (layer "B.Fab") (width 0.1))
     (fp_line (start -2.5 1.25) (end 2.5 1.25) (layer "B.Fab") (width 0.1))
-    (pad "1" smd roundrect (at -2.3125 0 90) (size 1.225 2.65) (layers "B.Cu" "B.Paste" "B.Mask") (roundrect_rratio 0.204082)
+    (pad "1" smd roundrect (at -2.3125 0 90) (size 1.225 2.65) (layers "B.Cu" "B.Paste" "B.Mask") (roundrect_rratio 0.2040816327)
       (net 61 "Net-(IC3-Pad27)") (pintype "passive"))
-    (pad "2" smd roundrect (at 2.3125 0 90) (size 1.225 2.65) (layers "B.Cu" "B.Paste" "B.Mask") (roundrect_rratio 0.204082)
+    (pad "2" smd roundrect (at 2.3125 0 90) (size 1.225 2.65) (layers "B.Cu" "B.Paste" "B.Mask") (roundrect_rratio 0.2040816327)
       (net 3 "GND") (pintype "passive"))
     (model "${KICAD6_3DMODEL_DIR}/Resistor_SMD.3dshapes/R_2010_5025Metric.wrl"
